File: hw/display.sch (KiCad schematic (older format))
At the start: 20 parts, among them J1 IDC_02X03, J2 SWD_01X04, Q1 AO3400A, U1 RC1602B, U2 STM32F042F6Px

Commit message: changed potentiometers link
Parts:
- RV1: symbol Device:POT -> Device:R_POT
Changed lines of the file:
@@
 	2650 4150 2650 3550
 $Comp
-L Device:POT RV1
+L Device:R_POT RV1
 U 1 1 5AE66D20
 P 3350 3950
