File: hw/display.kicad_pcb (KiCad board)
At the start: 2 copper layers, 81 x 37 mm, 20 parts, among them J1 IDC_02X03, J2 SWD_01X04, Q1 AO3400A, U1 RC1602B, U2 STM32F042F6Px

Commit message: updated pcb
Parts:
- added G***: LOGO, KLIB_Logo:wykys_skill, F.Cu at (148.0, 70.0)
- added REF**: Fiducial_Pad_1mm_Outer_2mm, KLIB_Mechanical:Fiducial_Pad_1mm_Outer_2mm, F.Cu at (156.0, 68.0)
- added REF**: Fiducial_Pad_1mm_Outer_2mm, KLIB_Mechanical:Fiducial_Pad_1mm_Outer_2mm, F.Cu at (156.0, 91.0)
- added REF**: Fiducial_Pad_1mm_Outer_2mm, KLIB_Mechanical:Fiducial_Pad_1mm_Outer_2mm, F.Cu at (90.0, 68.0)
- moved J1 45.5 mm to (96.0, 74.8)
- moved C5 45.0 mm to (89.2, 85.2), turned to 180 degrees
- moved C4 42.4 mm to (89.2, 88.2), turned to 180 degrees
- moved Q1 9.45 mm to (118.2, 89.0)
- moved C2 8.62 mm to (100.8, 85.8)
- moved R1 8.62 mm to (100.8, 83.8)
- moved J2 8.31 mm to (112.0, 74.8)
- moved U2 7.72 mm to (108.8, 85.0)
- moved C1 7.35 mm to (116.5, 84.8)
- moved C3 3.78 mm to (89.2, 90.2), turned to 180 degrees
- moved RV1 1.95 mm to (140.2, 79.0)
- moved R3 1.58 mm to (136.0, 84.2)
- moved R2 1.12 mm to (136.0, 79.0)
- moved JP2 0.50 mm to (136.0, 88.2)
Connections:
- U2 pad 8: /LCD_TX -> /LCD_UART_TX
- U2 pad 9: /LCD_RX -> /LCD_UART_RX
Routing:
- net +3V3: track 0.00 -> 139.5 mm
- net Net-(JP1-Pad1): track 0.00 -> 131.8 mm, vias 0 -> 1
- net /RS: track 0.00 -> 27.7 mm, vias 0 -> 1
- net /DB7: track 0.00 -> 26.9 mm, vias 0 -> 1
- net /R~W: track 0.00 -> 26.5 mm, vias 0 -> 1
- net /E: track 0.00 -> 25.4 mm, vias 0 -> 1
- net /LCD_UART_RX: track 0.00 -> 24.1 mm, vias 0 -> 1
- net /LCD_UART_TX: track 0.00 -> 23.5 mm, vias 0 -> 1
- net /DB6: track 0.00 -> 23.3 mm, vias 0 -> 1
- net /~RST: track 0.00 -> 20.4 mm
- net Net-(JP1-Pad2): track 0.00 -> 17.1 mm
- net /DB1: track 0.00 -> 15.1 mm
- net /DB0: track 0.00 -> 14.8 mm
- net Net-(Q1-Pad3): track 0.00 -> 14.0 mm, vias 0 -> 1
- net /DB5: track 0.00 -> 13.8 mm
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- added copper zone on B.Cu, net GND
- added copper zone on F.Cu, net GND
Other:
- board text added: "DISPLAY V2"

Commit message: updated pcb layout
Routing:
- net Net-(JP1-Pad1): track 131.8 -> 125.0 mm
- net /RS: track 27.7 -> 32.9 mm
- net /DB2: track 13.7 -> 9.61 mm
- net /R~W: track 26.5 -> 28.2 mm
- net +3V3: track 139.5 -> 140.4 mm
- net /LCD_UART_RX: track 24.1 -> 23.4 mm
- net /SWCLK: track 10.1 -> 10.7 mm
- net /SWDIO: track 11.8 -> 12.4 mm
- net GND: vias 28 -> 29
