File: hw/display.kicad_pcb (KiCad board)
At the start: 2 copper layers, 81 x 37 mm, 24 parts, among them J1 IDC_02X03, J2 SWD_01X04, Q1 AO3400A, U1 RC1602B, U2 STM32F042F6Px

Commit message: updated layout
Routing:
- net Net-(JP1-Pad1): track 125.0 -> 127.8 mm, vias 1 -> 3
Changed lines of the file:
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@@
     (thickness 1.6)
     (drawings 5)
-    (tracks 255)
+    (tracks 258)
     (zones 0)
     (modules 24)
@@
   )
   (setup
-    (last_trace_width 0.25)
+    (last_trace_width 0.8)
     (user_trace_width 0.5)
     (user_trace_width 0.8)
@@
   (segment (start 92.94 93) (end 92.94 95.5) (width 1) (layer F.Cu) (net 1))
   (segment (start 95.96 72.25) (end 95.96 74.79) (width 1) (layer F.Cu) (net 1))
+  (segment (start 123 86.45) (end 123 84.575) (width 0.8) (layer F.Cu) (net 2))
+  (segment (start 123 85.524996) (end 123 86.45) (width 0.8) (layer B.Cu) (net 2))
+  (segment (start 123 85.524996) (end 123 84.575) (width 0.8) (layer F.Cu) (net 2))
+  (via (at 123 84.575) (size 0.8) (drill 0.4) (layers F.Cu B.Cu) (net 2))
+  (segment (start 123 67) (end 123 85.524996) (width 0.8) (layer B.Cu) (net 2))
+  (via (at 123 85.524996) (size 0.8) (drill 0.4) (layers F.Cu B.Cu) (net 2))
+  (segment (start 123 86.55) (end 123 86.45) (width 0.8) (layer F.Cu) (net 2))
+  (via (at 123 86.45) (size 0.8) (drill 0.4) (layers F.Cu B.Cu) (net 2))
+  (segment (start 124.7 88.25) (end 123 86.55) (width 0.8) (layer F.Cu) (net 2))
   (segment (start 122.07 67) (end 123 67) (width 1) (layer B.Cu) (net 2))
   (segment (start 123 67) (end 137 67) (width 1) (layer B.Cu) (net 2))
-  (segment (start 123 67.93) (end 123 67) (width 0.8) (layer B.Cu) (net 2))
-  (segment (start 123 84.76) (end 123 67.93) (width 0.8) (layer B.Cu) (net 2))
-  (segment (start 123 85.325685) (end 123 84.76) (width 0.8) (layer F.Cu) (net 2))
-  (segment (start 123 86.55) (end 123 85.325685) (width 0.8) (layer F.Cu) (net 2))
-  (segment (start 124.7 88.25) (end 123 86.55) (width 0.8) (layer F.Cu) (net 2))
-  (via (at 123 84.76) (size 0.8) (drill 0.4) (layers F.Cu B.Cu) (net 2))
   (segment (start 94.5 67) (end 122.07 67) (width 1) (layer B.Cu) (net 2))
   (segment (start 91.25 88.75) (end 91.25 70.25) (width 1) (layer B.Cu) (net 2))
